File: addons/energystorage_4MU_MID/addon_energystorage_4MU_MID.brd (EAGLE design)
At the start: 68 x 59.9 mm, 31 parts, among them IC1 74HC595D, IC2 74HC595D, Q1 BCP52

Commit message: [Application - out8 16A - bistable relay - 4TE - BOT] erc edited
Parts:
- SV1: value (none) -> B
Changed lines of the file:
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@@
 <attribute name="OC_NEWARK" value="unknown" x="55.626" y="24.834" size="1.778" layer="28" rot="MR270" display="off"/>
 </element>
-<element name="SV1" library="pinhead" package="2X13SMD" value="" x="32.512" y="29.152" smashed="yes" rot="R90">
+<element name="SV1" library="pinhead" package="2X13SMD" value="B" x="32.512" y="29.152" smashed="yes" rot="R90">
 <attribute name="NAME" x="31.242" y="10.991" size="1.016" layer="25" ratio="10"/>
-<attribute name="VALUE" x="38.227" y="12.642" size="1.27" layer="27" rot="R90"/>
 </element>
 <element name="Q1" library="transistor-pnp" package="SOT223" value="BCP52" x="15.494" y="22.04" smashed="yes" rot="R90">
