File: applications_din/out_8x_16A_bistab_4MU/out_8x_16A_bistab_4MU_v2.0.0/app_out_8x_16A_bistab_4MU_BOT_v2.0.0.brd (EAGLE design)
At the start: 86.3 x 67.3 mm, 31 parts, among them IC1 ULN2803, IC2 ULN2803, K1 HFE20-1, K2 HFE20-1, K3 HFE20-1, K4 HFE20-1, K5 HFE20-1, K6 HFE20-1, K7 HFE20-1, K8 HFE20-1

Commit message: [Application - out8 16A - bistable relay - 4TE - BOT] erc edited
Parts:
- JP2, SJ1: value (none) -> A
Changed lines of the file:
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@@
 <attribute name="OC_FARNELL" value="unknown" x="7.874" y="63.9445" size="1.778" layer="27" rot="R270" display="off"/>
 </element>
-<element name="JP2" library="pinhead" package="2X13SMD" value="" x="57.785" y="7.62" smashed="yes" rot="R180">
+<element name="JP2" library="pinhead" package="2X13SMD" value="A" x="57.785" y="7.62" smashed="yes" rot="R180">
 <attribute name="NAME" x="60.459728125" y="4.148665625" size="1.27" layer="25" ratio="10"/>
-<attribute name="VALUE" x="60.325" y="13.335" size="1.27" layer="27" rot="R180"/>
 </element>
 <element name="R1" library="rcl" package="M1206" value="680" x="22.352" y="9.652" smashed="yes" rot="MR90">
@@
 <attribute name="VALUE" x="63.754" y="12.065" size="1.27" layer="27" ratio="10" rot="R270"/>
 </element>
-<element name="SJ1" library="jumper" package="SJ" value="" x="22.352" y="3.81" smashed="yes" rot="R180">
+<element name="SJ1" library="jumper" package="SJ" value="A" x="22.352" y="3.81" smashed="yes" rot="R180">
 <attribute name="NAME" x="27.305" y="4.445" size="1.27" layer="25" ratio="10" rot="R180"/>
 <attribute name="VALUE" x="21.9519" y="3.81" size="0.02" layer="27" rot="R180"/>
@@
 <vertex x="82.55" y="28.067"/>
 <vertex x="84.709" y="28.067"/>
-<vertex x="84.709" y="33.782"/>
 </polygon>
 <polygon width="1.27" layer="16" thermals="no">
