File: modules_lpc1115_fm/IO-8x-fused-35x25-fm/IO-module-8x_fused_in-wall_35x25.sch (EAGLE design)
At the start: 87 parts, among them IC1 LPC1115, IC2 ATAES132A-SHEQ-T, Q2 ASFL, U1 EEPROM, X3 MICROMATCH-10

Commit message: [IOmodule8xUP] - some minor optimizations
corrected mixed up SWDIO / SWCLK labels
optimized some vias
optimized schematic
added ferrite values
Parts:
- FB10, FB3, FB4, FB5, FB6, FB7, FB8, FB9: value (none) -> 1.5kΩ@100MHz
- JP1: value B4B-PH-K-S -> 653005114822; device con-JST PH:B4B-PH-K-S -> Wurth_Connectors_WR-WTB:653005114822
Connections:
- net SWD_SWCLK: now also JP7.4, R17.2, TVS3.IO1; no longer JP7.2, R19.2, TVS3.IO2
- net SWD_SWDIO: now also JP7.2, R19.2, TVS3.IO2; no longer JP7.4, R17.2, TVS3.IO1
Other:
- note added: "Pins for stabilization and heat dissipation"

Commit message: [IOmodule8xUP] - breaking change of routing, I2C optimization
re-routed some IOs to other ARM pins
added 2nd alternative to connect I2C peripherals
Parts:
- removed LED2: red, led:LED3MM
- removed LED3: red SMD, led:LEDCHIPLED_1206
- added JP5: (no value), pinhead_dmx:PINHD-1X4
- JP1: value 653005114822 -> 62000411622; device Wurth_Connectors_WR-WTB:653005114822 -> Eagle_WR-WTB (rev22a):62000411622
Connections:
- net +3V3: now also JP5.1
- net GND: now also JP5.2
- net IO4: now also IC1.PIO0_7/CTS; no longer IC1.PIO3_5/CT16B1_CAP1/TXD
- net IO5: now also IC1.PIO3_5/CT16B1_CAP1/TXD; no longer IC1.PIO0_6/SCK0
- net IO7: now also IC1.PIO0_6/SCK0; no longer IC1.TDO/PIO1_1/AD2/CT32B1_MAT0
- net IO8: now also IC1.PIO2_9/CT32B0_CAP0; no longer IC1.TRST/PIO1_2/AD3/CT32B1_MAT1
- net N$41: no longer LED2.A, LED3.A
- net PROG: no longer LED2.C, LED3.C
- net SCL: now also JP5.3
- net SDA: now also JP5.4
Other:
- moved on the sheet: JP2, JP3, JP4, JP7, R17, R18, R19, R20, R23, R24, TVS3

Commit message: [IOmodule8xUP] - changed values to standard values
Parts:
- C1, C12, C15, C2, C20, C21: value 100n -> 100nF
- C11, C13: value 1µ -> 1uF
- C14, C9: value 10n -> 10nF
- C7: value 220p -> 220pF
- C8: value 100p -> 100pF
Other:
- moved on the sheet: C20, X3-1, X3-10, X3-2, X3-3, X3-4, X3-5, X3-6, X3-7, X3-8, X3-9
