File: modules_lpc1115_fm/IO-8x-fused-35x25-fm/IOmodule-8x_fused_35x25_fm.sch (EAGLE design)
At the start: 86 parts, among them IC1 LPC1115, IC2 ATAES132A-SHEQ-T, Q2 ASFL, U1 EEPROM, X3 MICROMATCH-10

Commit message: [IOmodule8xFM] parts re-arranged; pin assignement of I2C conn. corrected
Parts:
- C1, C11, C9: REICHELT X7R-G0805 10N -> (none)
- C12, C13, C15, C2: REICHELT X7R-G0805 100N -> (none)
- D31: device Diode:DIODE_DO-219-AB(SOD123F) -> microbuilder:DIODESOD-123
- D32, D33, D35, D36, D37, D38: value DIODE -> DDZ9684; device Diode:DIODE_DO-219-AB(SOD123F) -> microbuilder:DIODESOD-123
- D34: value PDZ3.3BGWJ -> DDZ9684; device Diode:DIODE_DO-219-AB(SOD123F) -> microbuilder:DIODESOD-123
- F17, F18, F19, F20, F21, F22, F23: value 0805L035 -> BSMD0805-005-33V
- F24: value 0805L050 -> BSMD0805-005-33V; device polyfuse-smd_10:0805L050 -> polyfuse-smd_10:0805L035
- LED1: device led:LEDCHIPLED_1206 -> led:LEDCHIPLED_0805; REICHELT SMD-LED 0805 RT -> (none)
- R1, R18, R20: REICHELT SMD-0805 3,30K -> (none)
- R14, R15: REICHELT SMD-0805 100K -> (none)
- R16: REICHELT SMD-0805 1,00K -> (none)
Connections:
- net +3V3: now also JP1.3; no longer JP1.2
- net GND: now also JP1.4; no longer JP1.1
- net SCL: now also JP1.1; no longer JP1.4
- net SDA: now also JP1.2; no longer JP1.3
Other:
- moved on the sheet: JP1

Commit message: [IOmodule8xFM] - switched RX / TX to 2,54 pin header added status LED
Parts:
- removed GND: TPTP11SQ, testpad:TPTP11SQ
- removed RXD: TPTP12R, testpad:TPTP12R
- removed TXD: TPTP12SQ, testpad:TPTP12SQ
- added JP6: (no value), pinhead_dmx:PINHD-1X2
- added LED2: (no value), led:LEDCHIPLED_0805
- added R10: 1k, rcl:R-EU_R0805
Connections:
- new net N$14: LED2.C, R10.2
- new net N$19: IC1.PIO3_3/RI/CT16B0_CAP0, R10.1
- net +3V3: now also LED2.A
- net DBG_RXD: now also JP6.2; no longer RXD.TP
- net DBG_TXD: now also JP6.1; no longer TXD.TP
- net GND: no longer GND.TP
Other:
- moved on the sheet: C1, C11, C12, C13, C14, C15, C2, C20, C21, C7, C8, C9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
